Commit message: Update

File: sa2000h_urdf_0416/urdf/sa2000h_urdf_0416.urdf (robot description, URDF)
Before this commit: robot sa2000h_urdf_0416, 9 links, 8 joints
Links:
- link base_link: geometry collision mesh filename=https://raw.githubusercontent.com/shine-tong/urdf/main/sa20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; visual mesh filename=https://raw.githubusercontent.com/shine-tong/urdf/main/sa20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
- link link1: geometry collision mesh filename=https://raw.githubusercontent.com/shine-tong/urdf/main/sa20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; visual mesh filename=https://raw.githubusercontent.com/shine-tong/urdf/main/sa20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
- link link2: geometry collision mesh filename=https://raw.githubusercontent.com/shine-tong/urdf/main/sa20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; visual mesh filename=https://raw.githubusercontent.com/shine-tong/urdf/main/sa20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
- link link3: geometry collision mesh filename=https://raw.githubusercontent.com/shine-tong/urdf/main/sa20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; visual mesh filename=https://raw.githubusercontent.com/shine-tong/urdf/main/sa20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
- link link4: geometry collision mesh filename=https://raw.githubusercontent.com/shine-tong/urdf/main/sa20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; visual mesh filename=https://raw.githubusercontent.com/shine-tong/urdf/main/sa20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
- link link5: geometry collision mesh filename=https://raw.githubusercontent.com/shine-tong/urdf/main/sa20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; visual mesh filename=https://raw.githubusercontent.com/shine-tong/urdf/main/sa20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
- link link6: geometry collision mesh filename=https://raw.githubusercontent.com/shine-tong/urdf/main/sa20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; visual mesh filename=https://raw.githubusercontent.com/shine-tong/urdf/main/sa20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
